File: minisumo/minisumo Partes 2/_autosave-minisumo Partes 2.kicad_sch (KiCad schematic)
At the start: 25 parts, among them J1 ENTRADA, J2 MOTOR1, J3 MOTOR2, J4 SENSOR ULTRASONICO, J5 SENSOR SHARP, J6 SENSOR SHARP, J7 SENSOR SHARP, J8 SENSOR CNY70, J9 SENSOR CNY70, SW1 SW_DPST_x2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

Commit message: 16/6
Parts:
- J1, J2, J3: footprint EESTN5:BORNERA2 -> EESTN5:BORNERA2_AZUL
Connections:
- net D15: now also J9.3 (Pin_3); no longer J8.3 (Pin_3)
- net D18: now also R7.2, R8.1
- net D19: no longer J9.3 (Pin_3)
- net D2: now also J4.2 (Pin_2)
- net D21: now also R3.2, R4.1
- net D22: no longer R7.2, R8.1
- net D32: no longer J4.2 (Pin_2)
- net D4: now also J8.3 (Pin_3)
- net VP: no longer R3.2, R4.1
Changed lines of the file:
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@@
 		)
 	)
-	(global_label "D32"
+	(global_label "D2"
 		(shape input)
 		(at 125.73 95.25 180)
@@
 		)
 		(property "Intersheetrefs" "${INTERSHEET_REFS}"
-			(at 119.0558 95.25 0)
+			(at 120.2653 95.25 0)
 			(effects
 				(font
@@
 		)
 	)
-	(global_label "D15"
+	(global_label "D4"
 		(shape input)
 		(at 135.89 142.24 180)
@@
 		)
 		(property "Intersheetrefs" "${INTERSHEET_REFS}"
-			(at 129.2158 142.24 0)
+			(at 130.4253 142.24 0)
 			(effects
 				(font
@@
 		)
 	)
-	(global_label "VP"
+	(global_label "D21"
 		(shape input)
 		(at 252.73 118.11 0)
@@
 		)
 		(property "Intersheetrefs" "${INTERSHEET_REFS}"
-			(at 258.0738 118.11 0)
+			(at 259.4042 118.11 0)
 			(effects
 				(font
@@
 		)
 	)
-	(global_label "D19"
+	(global_label "D15"
 		(shape input)
 		(at 165.1 142.24 180)
@@
 		)
 	)
-	(global_label "D22"
+	(global_label "D18"
 		(shape input)
 		(at 124.46 115.57 180)
@@
 			)
 		)
-		(property "Footprint" "EESTN5:BORNERA2"
+		(property "Footprint" "EESTN5:BORNERA2_AZUL"
 			(at 193.04 39.37 0)
 			(effects
@@
 			)
 		)
-		(property "Footprint" "EESTN5:BORNERA2"
+		(property "Footprint" "EESTN5:BORNERA2_AZUL"
 			(at 224.79 39.37 0)
 			(effects
@@
 			)
 		)
-		(property "Footprint" "EESTN5:BORNERA2"
+		(property "Footprint" "EESTN5:BORNERA2_AZUL"
 			(at 85.09 40.64 0)
 			(effects
