File: minisumo/minisumo Partes 2/minisumo Partes 2.kicad_pcb (KiCad board)
At the start: 2 copper layers, 25 parts, among them J1 ENTRADA, J2 MOTOR1, J3 MOTOR2, J4 SENSOR ULTRASONICO, J5 SENSOR SHARP, J6 SENSOR SHARP, J7 SENSOR SHARP, J8 SENSOR CNY70, J9 SENSOR CNY70, SW1 SW_DPST_x2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

Commit message: 16/6
Parts:
- removed U1: ESP32-DEVKITC-32E, ESP32-DEVKITC-32E (2):MODULE_ESP32-DEVKITC-32E
- added U4: ESP32-DEVKIT-V1, esp32 30 pines huella:MODULE_ESP32_DEVKIT_V1, F.Cu at (173.0, 74.0)
- J1, J2, J3: footprint EESTN5:BORNERA2 -> EESTN5:BORNERA2_AZUL
- moved J5 67.6 mm to (193.0, 92.5)
- moved R1 67.1 mm to (191.0, 82.5), turned to 180 degrees
- moved R2 65.2 mm to (191.2, 80.3), turned to 0 degrees
- moved R4 64.1 mm to (164.1, 56.5), turned to 0 degrees
- moved J7 61.4 mm to (152.1, 56.5), turned to 0 degrees
- moved R3 60.6 mm to (160.5, 56.5), turned to 0 degrees
- moved J2 55.9 mm to (182.5, 117.0), turned to 0 degrees
- moved J3 48.8 mm to (171.5, 117.0), turned to 0 degrees
- moved R6 47.4 mm to (161.5, 91.6)
- moved C4 46.6 mm to (182.5, 113.0), turned to 0 degrees
- moved J6 44.7 mm to (152.0, 92.5)
- moved R5 44.4 mm to (159.2, 91.6), turned to 90 degrees
- moved C1 37.6 mm to (157.4, 99.0)
- moved C3 37.2 mm to (171.5, 113.0), turned to 0 degrees
- moved J4 36.8 mm to (179.5, 55.0), turned to 180 degrees
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Connections:
- net IO21 renamed D18
- net IO34 renamed D27
- net IO35 renamed D21
- net SENSOR_VN renamed VN
- J4 pad 2: IO19 -> D2
- J8 pad 3: IO15 -> D4
- J9 pad 3: IO23 -> D15
Routing:
- net VN: track 136.7 -> 6.73 mm
- net D4: track 0.00 -> 54.1 mm
- net D15: track 0.00 -> 21.3 mm
- net +5V: track 137.5 -> 156.1 mm
- net +3V3: track 89.1 -> 73.7 mm
- net D27: track 6.32 -> 19.4 mm
- net Net-(J1-Pin_1): track 20.5 -> 9.51 mm
- net IO19: track 9.33 -> 0.00 mm
- net VCC: track 28.6 -> 37.5 mm
- net IO23: track 8.22 -> 0.00 mm
- net D2: track 0.00 -> 6.35 mm
- net IO15: track 6.11 -> 0.00 mm
- net GND: track 0.00 -> 6.00 mm
- net A1: track 19.0 -> 14.1 mm
- net B2: track 14.4 -> 9.75 mm
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